File: PCB/LAS_V2/AC_Monitor_sch.kicad_sch (KiCad schematic)
At the start: 8 parts, among them Q6 MMBT2222A, U5 EL357N

Commit message: Need to redo PCB again
Parts:
- added J12 (x2): Conn_01x02_Pin, Connector_PinHeader_1.27mm:PinHeader_1x02_P1.27mm_Vertical, symbol Connector:Conn_01x02_Pin
Connections:
- net OUT1: now also J12.1 (Pin_1); no longer R24.1, U5.4
- net at D11.1 (K), Q6.3 (C), R17.2: now also J12.2 (Pin_2); no longer U5.1
- new net: J12.2 (Pin_2), R24.1, U5.4
- new net: J12.1 (Pin_1), U5.1
Changed lines of the file:
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@@
     (stroke (width 0) (type default))
   )
-  (wire (pts (xy 90.17 39.37) (xy 102.87 39.37))
+  (wire (pts (xy 90.17 39.37) (xy 95.25 39.37))
     (stroke (width 0) (type default))
   )
@@
     (stroke (width 0) (type default))
   )
+  (wire (pts (xy 130.81 38.1) (xy 118.11 38.1))
+    (stroke (width 0) (type default))
+  )
   (wire (pts (xy 49.53 48.26) (xy 49.53 39.37))
     (stroke (width 0) (type default))
@@
     (stroke (width 0) (type default))
   )
-  (wire (pts (xy 129.54 38.1) (xy 118.11 38.1))
+  (wire (pts (xy 97.79 39.37) (xy 102.87 39.37))
+    (stroke (width 0) (type default))
+  )
+  (wire (pts (xy 138.43 38.1) (xy 133.35 38.1))
     (stroke (width 0) (type default))
   )
@@
     (effects (font (size 1.27 1.27)) (justify left))
   )
-  (hierarchical_label "OUT1" (shape input) (at 129.54 38.1 0) (fields_autoplaced)
+  (hierarchical_label "OUT1" (shape input) (at 138.43 38.1 0) (fields_autoplaced)
     (effects (font (size 1.27 1.27)) (justify left))
   )
@@
     )
   )
+  (symbol (lib_id "Connector:Conn_01x02_Pin") (at 97.79 34.29 270) (unit 1)
+    (in_bom yes) (on_board yes) (dnp no)
+    (property "Reference" "J12" (at 88.9 27.94 90)
+      (effects (font (size 1.27 1.27)) (justify left))
+    )
+    (property "Value" "Conn_01x02_Pin" (at 87.63 30.48 90)
+      (effects (font (size 1.27 1.27)) (justify left))
+    )
+    (property "Footprint" "Connector_PinHeader_1.27mm:PinHeader_1x02_P1.27mm_Vertical" (at 97.79 34.29 0)
+      (effects (font (size 1.27 1.27)) hide)
+    )
+    (property "Datasheet" "~" (at 97.79 34.29 0)
+      (effects (font (size 1.27 1.27)) hide)
+    )
+    (pin "1")
+    (pin "2")
+    (instances
+      (project "LAS_V2"
+        (path "/aadef4b8-3115-4a49-998f-828f2021a6b4"
+          (reference "J12") (unit 1)
+        )
+        (path "/aadef4b8-3115-4a49-998f-828f2021a6b4/e3f941ed-5575-4c88-95e0-e32be2fe0df6"
+          (reference "J14") (unit 1)
+        )
+      )
+    )
+  )
   (symbol (lib_id "Diode:ZMMxx") (at 82.55 49.53 270) (unit 1)
     (in_bom yes) (on_board yes) (dnp no)
@@
         )
       )
+    )
+  )
+  (symbol (lib_id "Connector:Conn_01x02_Pin") (at 133.35 33.02 270) (unit 1)
+    (in_bom yes) (on_board yes) (dnp no)
+    (property "Reference" "J12" (at 124.46 26.67 90)
+      (effects (font (size 1.27 1.27)) (justify left))
+    )
+    (property "Value" "Conn_01x02_Pin" (at 123.19 29.21 90)
+      (effects (font (size 1.27 1.27)) (justify left))
+    )
+    (property "Footprint" "Connector_PinHeader_1.27mm:PinHeader_1x02_P1.27mm_Vertical" (at 133.35 33.02 0)
+      (effects (font (size 1.27 1.27)) hide)
+    )
+    (property "Datasheet" "~" (at 133.35 33.02 0)
+      (effects (font (size 1.27 1.27)) hide)
+    )
+    (pin "1")
+    (pin "2")
+    (instances
+      (project "LAS_V2"
+        (path "/aadef4b8-3115-4a49-998f-828f2021a6b4"
+          (reference "J12") (unit 1)
+        )
+        (path "/aadef4b8-3115-4a49-998f-828f2021a6b4/e3f941ed-5575-4c88-95e0-e32be2fe0df6"
+          (reference "J13") (unit 1)
+        )
+      )

Commit message: Final Changes to PCB, more code for gateway
Parts:
- J12: footprint Connector_PinHeader_1.27mm:PinHeader_1x02_P1.27mm_Vertical -> Connector_PinHeader_2.54mm:PinHeader_1x02_P2.54mm_Vertical
- R17: footprint Resistor_THT:R_Axial_DIN0617_L17.0mm_D6.0mm_P25.40mm_Horizontal -> Resistor_THT:R_Axial_DIN0617_L17.0mm_D6.0mm_P20.32mm_Horizontal
Changed lines of the file:
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@@
       (effects (font (size 1.27 1.27)) (justify left))
     )
-    (property "Footprint" "Connector_PinHeader_1.27mm:PinHeader_1x02_P1.27mm_Vertical" (at 97.79 34.29 0)
+    (property "Footprint" "Connector_PinHeader_2.54mm:PinHeader_1x02_P2.54mm_Vertical" (at 97.79 34.29 0)
       (effects (font (size 1.27 1.27)) hide)
     )
@@
       (effects (font (size 1.27 1.27)))
     )
-    (property "Footprint" "Resistor_THT:R_Axial_DIN0617_L17.0mm_D6.0mm_P25.40mm_Horizontal" (at 73.66 39.37 0)
+    (property "Footprint" "Resistor_THT:R_Axial_DIN0617_L17.0mm_D6.0mm_P20.32mm_Horizontal" (at 73.66 39.37 0)
       (effects (font (size 1.27 1.27)) hide)
     )
@@
       (effects (font (size 1.27 1.27)) (justify left))
     )
-    (property "Footprint" "Connector_PinHeader_1.27mm:PinHeader_1x02_P1.27mm_Vertical" (at 133.35 33.02 0)
+    (property "Footprint" "Connector_PinHeader_2.54mm:PinHeader_1x02_P2.54mm_Vertical" (at 133.35 33.02 0)
       (effects (font (size 1.27 1.27)) hide)
     )
