File: PCB/LAS_V2/LAS_V2.kicad_pcb (KiCad board)
At the start: 2 copper layers, 95 x 95 mm, 63 parts, among them J1 Screw_Terminal_01x04, J2 Conn_01x03_Pin, J3 Conn_01x05_Socket, J4 Conn_01x22_Socket, J5 Conn_01x22_Socket, J6 Conn_01x02_Pin, J7 USB_C_Receptacle_USB2.0, J8 Conn_01x05, K1 SRD-05VDC-SL-C, Q1 MMBT2222A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

Commit message: Need to redo PCB again
Parts:
- removed SW1, SW2: SW_Push, Connector_PinHeader_1.27mm:PinHeader_1x02_P1.27mm_Vertical
- added J10: Conn_01x02_Pin, Connector_PinHeader_1.27mm:PinHeader_1x02_P1.27mm_Vertical, F.Cu at (131.3, 73.8)
- added J11: Conn_01x02_Pin, Connector_PinHeader_1.27mm:PinHeader_1x02_P1.27mm_Vertical, F.Cu at (134.6, 106.3)
- added J12: Conn_01x02_Pin, Connector_PinHeader_1.27mm:PinHeader_1x02_P1.27mm_Vertical, F.Cu at (118.8, 56.2)
- added J13: Conn_01x02_Pin, Connector_PinHeader_1.27mm:PinHeader_1x02_P1.27mm_Vertical, F.Cu at (151.6, 107.9)
- added J14: Conn_01x02_Pin, Connector_PinHeader_1.27mm:PinHeader_1x02_P1.27mm_Vertical, F.Cu at (151.2, 116.7)
- added J9: Conn_01x02_Pin, Connector_PinHeader_1.27mm:PinHeader_1x02_P1.27mm_Vertical, F.Cu at (167.0, 87.2)
- moved R3 18.5 mm to (136.9, 122.0), turned to -90 degrees
- moved C6 16.1 mm to (134.6, 122.0), turned to -90 degrees
- moved D8 11.9 mm to (178.2, 131.2)
- moved U2 11.0 mm to (134.6, 115.0), turned to 90 degrees
- moved D1 7.53 mm to (128.9, 106.9), turned to -90 degrees
- moved D6 4.29 mm to (201.2, 101.6)
- moved J6 4.29 mm to (198.4, 92.4)
- moved Q1 4.29 mm to (201.2, 97.0)
- moved R8 4.29 mm to (204.3, 101.6)
- moved R9 4.29 mm to (202.2, 93.1)
- moved D7 4.29 mm to (198.3, 101.7)
- moved R4 4.02 mm to (131.6, 107.1), turned to -90 degrees
- moved R13 3.00 mm to (186.0, 61.4)
- moved R14 3.00 mm to (189.0, 61.5), turned to 90 degrees
- moved C8 1.60 mm to (188.7, 74.5), turned to 90 degrees
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Connections:
- C6 pad 1: /+3.3V -> Net-(J11-Pin_2)
- J1 pad 2: /NC1 -> unconnected-(J1-Pin_2-Pad2)
- R24 pad 1: /AC_Mon_1 -> Net-(J13-Pin_2)
- TP2 pad 1: /+3.3V -> Net-(J11-Pin_2)
- U2 pad 2: /+3.3V -> Net-(J11-Pin_2)
- U3 pad 16: /+3.3V -> /VBus
- U5 pad 1: Net-(D11-K) -> Net-(J14-Pin_1)
- U5 pad 4: /AC_Mon_1 -> Net-(J13-Pin_2)
Routing:
- net /VBus: track 16.8 -> 292.0 mm, vias 0 -> 8
- net /+3.3V: track 0.00 -> 142.0 mm, vias 0 -> 4
- net /GPIO6: track 0.00 -> 78.6 mm, vias 0 -> 1
- net /CHIP_PU: track 0.00 -> 77.5 mm
- net /GPIO4: track 0.00 -> 64.3 mm, vias 0 -> 1
- net /BOOT_SEL: track 0.00 -> 57.1 mm, vias 0 -> 2
- net /TXD0: track 0.00 -> 47.0 mm, vias 0 -> 1
- net /AC_Mon_1: track 2.36 -> 49.2 mm, vias 0 -> 1
- net /RXD0: track 0.00 -> 45.1 mm, vias 0 -> 1
- net /DIN_3.3: track 0.00 -> 43.1 mm, vias 0 -> 1
- net Net-(J11-Pin_2): track 0.00 -> 35.1 mm
- net /GPIO19: track 0.00 -> 31.3 mm, vias 0 -> 1
- net /GPIO20: track 0.00 -> 26.7 mm, vias 0 -> 1
- net /GPIO14: track 0.00 -> 21.0 mm
- net /GPIO13: track 0.00 -> 19.1 mm
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Other:
- board text added: "3.3V"
- board text added: "3.3V BRIDGE"
- board text added: "5V"
- board text added: "5V to 3.3V"
- board text added: "AC Monitor"
- board text added: "FBR"
- board text added: "GND"
- board text added: "J13 - After Opt J14 - Before Opt"
- board text added: "J8: 5V RX TX D+ D-"
- board text added: "N0 | X | LIVE | NEUT ^Don't mess it up"
- board text added: "PU"
- board text added: "RFID Reader"
- board text added: "Relay Controls"
- board text added: "TX"

Commit message: Updated rme
Parts:
- moved D4 70.7 mm to (115.5, 127.8), turned to 90 degrees
- moved R28 68.2 mm to (121.0, 121.3), turned to 90 degrees
- moved Q6 65.4 mm to (117.5, 121.7), turned to 180 degrees
- moved R29 61.9 mm to (114.0, 121.3), turned to -90 degrees
- moved R1 61.8 mm to (117.5, 118.3), turned to 0 degrees
- moved J12 59.7 mm to (118.0, 115.8), turned to -90 degrees
- moved C6 14.2 mm to (133.8, 136.2)
- moved D1 14.2 mm to (128.2, 121.0)
- moved U2 14.2 mm to (133.8, 129.1)
- moved J11 14.2 mm to (133.8, 120.5)
- moved R3 14.2 mm to (136.2, 136.1)
- moved R4 14.2 mm to (130.9, 121.2)
- moved R13 14.1 mm to (181.3, 74.7)
- moved J8 14.1 mm to (192.9, 84.3)
- moved C7 14.1 mm to (192.5, 76.8)
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Routing:
- net /CHIP_PU: track 77.5 -> 141.5 mm, vias 0 -> 8
- net /DIN_3.3: track 43.1 -> 69.3 mm, vias 1 -> 3
- net Net-(J11-Pin_2): track 35.1 -> 54.8 mm, vias 0 -> 1
- net /BOOT_SEL: track 57.1 -> 43.2 mm
- net /+3.3V: track 142.0 -> 154.3 mm, vias 4 -> 1
- net /TX_RFID: track 12.8 -> 21.6 mm
- net /GPIO4: track 64.3 -> 72.3 mm, vias 1 -> 3
- net Net-(D8-+): track 14.8 -> 7.55 mm
- net /NEUTRAL: track 43.9 -> 37.6 mm
- net GND: track 0.00 -> 6.20 mm, vias 17 -> 19
- net /RXD0: track 45.1 -> 49.2 mm
- net /GPIO1: track 15.9 -> 12.6 mm
- net Net-(D6-K): track 26.6 -> 23.8 mm
- net /GPIO2: track 18.8 -> 16.2 mm
- net /GPIO6: track 78.6 -> 76.6 mm
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- added copper zone on B.Cu, net GND
- added copper zone on F.Cu, net GND
Other:
- board size 95 x 95 mm -> 97.5 x 75.5 mm
- board text added: "ON"

Commit message: Final Changes to PCB, more code for gateway
Parts:
- removed C8: 1uF, Capacitor_SMD:C_0603_1608Metric
- removed R1, R3: 0, Resistor_SMD:R_0603_1608Metric
- added D9: WS2812B, LED_SMD:LED_WS2812B_PLCC4_5.0x5.0mm_P3.2mm, F.Cu at (115.5, 138.4)
- J1: value Screw_Terminal_01x04 -> Screw_Terminal_01x03; footprint TerminalBlock_Phoenix:TerminalBlock_Phoenix_MKDS-1,5-4-5.08_1x04_P5.08mm_Horizontal -> TerminalBlock:TerminalBlock_bornier-3_P5.08mm
- J10, J11, J12, J13, J14, J6, J9: footprint Connector_PinHeader_1.27mm:PinHeader_1x02_P1.27mm_Vertical -> Connector_PinHeader_2.54mm:PinHeader_1x02_P2.54mm_Vertical
- J2: footprint Connector_PinHeader_1.27mm:PinHeader_1x03_P1.27mm_Vertical -> Connector_PinHeader_2.54mm:PinHeader_1x03_P2.54mm_Vertical
- J3: footprint Connector_PinHeader_1.27mm:PinHeader_1x05_P1.27mm_Vertical -> Connector_PinHeader_2.54mm:PinHeader_1x05_P2.54mm_Vertical
- J4, J5: footprint Connector_PinHeader_1.27mm:PinHeader_1x22_P1.27mm_Vertical -> Connector_PinHeader_2.54mm:PinHeader_1x22_P2.54mm_Vertical
- R17: footprint Resistor_THT:R_Axial_DIN0617_L17.0mm_D6.0mm_P25.40mm_Horizontal -> Resistor_THT:R_Axial_DIN0617_L17.0mm_D6.0mm_P20.32mm_Horizontal
- moved D1 24.8 mm to (144.8, 139.4), turned to 90 degrees
- moved J13 24.4 mm to (149.3, 132.2)
- moved J14 23.4 mm to (149.5, 140.0)
- moved R4 20.2 mm to (145.0, 135.6)
- moved Q4 19.4 mm to (168.0, 135.3)
- moved D11 19.4 mm to (172.2, 133.3)
- moved U5 19.4 mm to (155.1, 133.4)
- moved R20 19.4 mm to (163.5, 136.2)
- moved R21 19.4 mm to (159.8, 136.2)
- moved R17 19.3 mm to (178.6, 141.2)
- moved R24 19.1 mm to (153.1, 127.9), turned to 180 degrees
- moved J9 16.8 mm to (168.2, 104.0)
- moved C2 16.4 mm to (169.0, 101.1)
- moved J11 12.2 mm to (140.1, 131.0), turned to -90 degrees
- moved U2 9.80 mm to (138.4, 137.8)
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Connections:
- C7 pad 1: /VBus -> /VCC_5V
- D4 pad 1: /VBus -> /VCC_5V
- D4 pad 2: unconnected-(D4-DOUT-Pad2) -> Net-(D4-DOUT)
- D7 pad 1: /VBus -> /VCC_5V
- J1 pad 1: /N01 -> /NEUTRAL
- J1 pad 2: unconnected-(J1-Pin_2-Pad2) -> /N01
- J2 pad 2: /VBus -> /VCC_5V
- J3 pad 5: /VBus -> /VCC_5V
- J7 pad A4: /VBus -> /VCC_5V
- J7 pad A9: /VBus -> /VCC_5V
- J7 pad B4: /VBus -> /VCC_5V
- J7 pad B9: /VBus -> /VCC_5V
- J8 pad 5: /VBus -> /VCC_5V
- K1 pad 2: /VBus -> /VCC_5V
- R27 pad 1: /VBus -> /VCC_5V
- R29 pad 1: /VBus -> /VCC_5V
- R8 pad 1: /VBus -> /VCC_5V
- TP1 pad 1: /VBus -> /VCC_5V
- U2 pad 3: Net-(U2-VI) -> /VCC_5V
- U3 pad 16: /VBus -> /+3.3V
- U3 pad 4: Net-(U3-V3) -> /+3.3V
Routing:
- net /VCC_5V: track 0.00 -> 357.5 mm, vias 0 -> 7
- net /VBus: track 293.0 -> 0.00 mm, vias 9 -> 0
- net /+3.3V: track 154.3 -> 249.0 mm, vias 1 -> 3
- net /CHIP_PU: track 141.5 -> 71.9 mm, vias 8 -> 1
- net /BOOT_SEL: track 43.2 -> 75.8 mm
- net /NEUTRAL: track 37.6 -> 8.10 mm, vias 0 -> 1
- net /AC_Mon_1: track 49.2 -> 70.2 mm, vias 1 -> 0
- net /GPIO18: track 12.3 -> 32.5 mm, vias 0 -> 2
- net /GPIO21: track 11.6 -> 29.5 mm
- net /GPIO47: track 10.1 -> 26.5 mm
- net /GPIO14: track 21.0 -> 36.6 mm
- net /GPIO48: track 8.55 -> 23.4 mm
- net /GPIO13: track 19.1 -> 33.6 mm
- net /GPIO45: track 5.87 -> 20.3 mm
- net /GPIO35: track 4.10 -> 17.2 mm
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Other:
- board size 97.5 x 75.5 mm -> 97.5 x 79.6 mm
- board text added: "MIKHAIL RUSSELL EEE4022S LAS V2"
- board text added: "NEUT | NO | LIVE | ^Don't mess it up"
- board text removed: "N0 | X | LIVE | NEUT ^Don't mess it up"
