File: PCB/LAS_V2/LAS_V2.kicad_sch (KiCad schematic)
At the start: 22 parts, among them J1 Screw_Terminal_01x04, J2 Conn_01x03_Pin, J3 Conn_01x05_Socket, J4 Conn_01x22_Socket, J5 Conn_01x22_Socket, SW1 SW_Push, SW2 SW_Push, U1 ESP32-S3-WROOM-1, U2 AMS1117-3.3

Commit message: Need to redo PCB again
Parts:
- removed R1: 0, Resistor_SMD:R_0603_1608Metric, symbol Device:R_Small_US
- removed SW1, SW2: SW_Push, Connector_PinHeader_1.27mm:PinHeader_1x02_P1.27mm_Vertical, symbol Switch:SW_Push
- added J10, J11, J12, J9: Conn_01x02_Pin, Connector_PinHeader_1.27mm:PinHeader_1x02_P1.27mm_Vertical, symbol Connector:Conn_01x02_Pin
Connections:
- net +3.3V: now also J11.1 (Pin_1); no longer C4.1, TP2.1, U2.2 (VO)
- net BOOT_SEL: now also J9.1 (Pin_1)
- net CHIP_PU: now also J10.1 (Pin_1)
- net DIN_3.3: now also J12.1 (Pin_1)
- net GND: now also J10.2 (Pin_2), J9.2 (Pin_2)
- net LEDs/DIN: now also J12.2 (Pin_2)
- net NC1: no longer J1.2 (Pin_2)
- new net: C4.1, J11.2 (Pin_2), TP2.1, U2.2 (VO)
- no-connect marks 4 -> 5
Other:
- note added: "Conn for RD6300"
- moved on the sheet: C4, D1, J1, J2, J3, R3, TP1, TP2, U2

Commit message: Final Changes to PCB, more code for gateway
Parts:
- removed J1: Screw_Terminal_01x04, TerminalBlock_Phoenix:TerminalBlock_Phoenix_MKDS-1,5-4-5.08_1x04_P5.08mm_Horizontal, symbol Connector:Screw_Terminal_01x04
- removed R3: 0, Resistor_SMD:R_0603_1608Metric, symbol Device:R_Small_US
- added J1: Screw_Terminal_01x03, TerminalBlock:TerminalBlock_bornier-3_P5.08mm, symbol Connector:Screw_Terminal_01x03
- J10, J11, J12, J9: footprint Connector_PinHeader_1.27mm:PinHeader_1x02_P1.27mm_Vertical -> Connector_PinHeader_2.54mm:PinHeader_1x02_P2.54mm_Vertical
- J2: footprint Connector_PinHeader_1.27mm:PinHeader_1x03_P1.27mm_Vertical -> Connector_PinHeader_2.54mm:PinHeader_1x03_P2.54mm_Vertical
- J3: footprint Connector_PinHeader_1.27mm:PinHeader_1x05_P1.27mm_Vertical -> Connector_PinHeader_2.54mm:PinHeader_1x05_P2.54mm_Vertical
- J4, J5: footprint Connector_PinHeader_1.27mm:PinHeader_1x22_P1.27mm_Vertical -> Connector_PinHeader_2.54mm:PinHeader_1x22_P2.54mm_Vertical
Connections:
- net LIVE: now also J1.3 (Pin_3)
- net N01: now also J1.2 (Pin_2)
- net NEUTRAL: now also J1.1 (Pin_1)
- net VCC_5V: now also U2.3 (VI)
- no-connect marks 5 -> 4
Other:
- sheet USB Interface ports: added none; removed VBus
Changed lines of the file:
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@@
   )
   (no_connect (at 46.99 185.42))
-  (no_connect (at 30.48 54.61))
   (no_connect (at 46.99 187.96))
   (no_connect (at 264.16 106.68))
@@
     (stroke (width 0) (type default))
   )
-  (wire (pts (xy 30.48 49.53) (xy 40.64 49.53))
-    (stroke (width 0) (type default))
-  )
-  (wire (pts (xy 41.91 57.15) (xy 30.48 57.15))
+  (wire (pts (xy 30.48 54.61) (xy 40.64 54.61))
+    (stroke (width 0) (type default))
+  )
+  (wire (pts (xy 41.91 52.07) (xy 30.48 52.07))
     (stroke (width 0) (type default))
   )
@@
     (stroke (width 0) (type default))
   )
-  (wire (pts (xy 214.63 22.86) (xy 215.9 22.86))
-    (stroke (width 0) (type default))
-  )
   (wire (pts (xy 245.11 113.03) (xy 236.22 113.03))
     (stroke (width 0) (type default))
@@
     (stroke (width 0) (type default))
   )
-  (wire (pts (xy 220.98 22.86) (xy 223.52 22.86))
+  (wire (pts (xy 214.63 22.86) (xy 223.52 22.86))
     (stroke (width 0) (type default))
   )
@@
     (stroke (width 0) (type default))
   )
-  (wire (pts (xy 106.68 110.49) (xy 109.22 110.49))
-    (stroke (width 0) (type default))
-  )
   (wire (pts (xy 212.09 22.86) (xy 214.63 22.86))
     (stroke (width 0) (type default))
@@
     (stroke (width 0) (type default))
   )
-  (wire (pts (xy 41.91 52.07) (xy 30.48 52.07))
+  (wire (pts (xy 41.91 49.53) (xy 30.48 49.53))
     (stroke (width 0) (type default))
   )
@@
     (effects (font (size 1.27 1.27)) (justify right bottom))
   )
-  (label "NEUTRAL" (at 40.64 49.53 0) (fields_autoplaced)
+  (label "NEUTRAL" (at 40.64 54.61 0) (fields_autoplaced)
     (effects (font (size 1.27 1.27)) (justify left bottom))
   )
@@
     (effects (font (size 1.27 1.27)) (justify left bottom))
   )
-  (label "VBus" (at 109.22 110.49 0) (fields_autoplaced)
-    (effects (font (size 1.27 1.27)) (justify left bottom))
-  )
   (label "DIN_3.3" (at 35.56 154.94 180) (fields_autoplaced)
     (effects (font (size 1.27 1.27)) (justify right bottom))
@@
     (effects (font (size 1.27 1.27)) (justify left bottom))
   )
-  (label "N01" (at 41.91 57.15 0) (fields_autoplaced)
+  (label "N01" (at 41.91 52.07 0) (fields_autoplaced)
     (effects (font (size 1.27 1.27)) (justify left bottom))
   )
@@
     (effects (font (size 1.27 1.27)) (justify right bottom))
   )
-  (label "LIVE" (at 41.91 52.07 0) (fields_autoplaced)
+  (label "LIVE" (at 41.91 49.53 0) (fields_autoplaced)
     (effects (font (size 1.27 1.27)) (justify left bottom))
   )
@@
       (effects (font (size 1.27 1.27)))
     )
-    (property "Footprint" "Connector_PinHeader_1.27mm:PinHeader_1x05_P1.27mm_Vertical" (at 41.91 185.42 0)
+    (property "Footprint" "Connector_PinHeader_2.54mm:PinHeader_1x05_P2.54mm_Vertical" (at 41.91 185.42 0)
       (effects (font (size 1.27 1.27)) hide)
     )
@@
     )
   )
-  (symbol (lib_id "Device:R_Small_US") (at 218.44 22.86 270) (unit 1)
-    (in_bom yes) (on_board yes) (dnp no)
-    (property "Reference" "R3" (at 214.63 25.4 90)
-      (effects (font (size 1.27 1.27)))
-    )
-    (property "Value" "0" (at 222.25 25.4 90)
-      (effects (font (size 1.27 1.27)))
-    )
-    (property "Footprint" "Resistor_SMD:R_0603_1608Metric" (at 218.44 22.86 0)
-      (effects (font (size 1.27 1.27)) hide)
-    )
-    (property "Datasheet" "~" (at 218.44 22.86 0)
-      (effects (font (size 1.27 1.27)) hide)
-    )
-    (pin "1")
-    (pin "2")
-    (instances
-      (project "LAS_V2"
-        (path "/aadef4b8-3115-4a49-998f-828f2021a6b4"
-          (reference "R3") (unit 1)
-        )
-      )
-    )
-  )
   (symbol (lib_id "Connector:Conn_01x02_Pin") (at 50.8 165.1 90) (unit 1)
     (in_bom yes) (on_board yes) (dnp no)
@@
       (effects (font (size 1.27 1.27)) (justify left))
     )
-    (property "Footprint" "Connector_PinHeader_1.27mm:PinHeader_1x02_P1.27mm_Vertical" (at 50.8 165.1 0)
+    (property "Footprint" "Connector_PinHeader_2.54mm:PinHeader_1x02_P2.54mm_Vertical" (at 50.8 165.1 0)
       (effects (font (size 1.27 1.27)) hide)
     )
@@
       (effects (font (size 1.27 1.27)) (justify right))
     )
-    (property "Footprint" "Connector_PinHeader_1.27mm:PinHeader_1x02_P1.27mm_Vertical" (at 156.21 142.24 0)
+    (property "Footprint" "Connector_PinHeader_2.54mm:PinHeader_1x02_P2.54mm_Vertical" (at 156.21 142.24 0)
       (effects (font (size 1.27 1.27)) hide)
     )
@@
       (effects (font (size 1.27 1.27)) (justify left))
     )
-    (property "Footprint" "Connector_PinHeader_1.27mm:PinHeader_1x22_P1.27mm_Vertical" (at 269.24 78.74 0)
+    (property "Footprint" "Connector_PinHeader_2.54mm:PinHeader_1x22_P2.54mm_Vertical" (at 269.24 78.74 0)
       (effects (font (size 1.27 1.27)) hide)
     )
@@
     )
   )
+  (symbol (lib_id "Connector:Screw_Terminal_01x03") (at 25.4 52.07 180) (unit 1)
+    (in_bom yes) (on_board yes) (dnp no) (fields_autoplaced)
+    (property "Reference" "J1" (at 25.4 44.45 0)
+      (effects (font (size 1.27 1.27)))
+    )
+    (property "Value" "Screw_Terminal_01x03" (at 25.4 46.99 0)
+      (effects (font (size 1.27 1.27)))
+    )
+    (property "Footprint" "TerminalBlock:TerminalBlock_bornier-3_P5.08mm" (at 25.4 52.07 0)
+      (effects (font (size 1.27 1.27)) hide)
+    )
+    (property "Datasheet" "~" (at 25.4 52.07 0)
+      (effects (font (size 1.27 1.27)) hide)
+    )
+    (pin "1")
+    (pin "2")
+    (pin "3")
+    (instances
+      (project "LAS_V2"
+        (path "/aadef4b8-3115-4a49-998f-828f2021a6b4"
+          (reference "J1") (unit 1)
+        )
+      )
+    )
+  )
   (symbol (lib_id "Device:R_Small_US") (at 130.81 53.34 0) (unit 1)
     (in_bom yes) (on_board yes) (dnp no)
@@
         (path "/aadef4b8-3115-4a49-998f-828f2021a6b4"
           (reference "R2") (unit 1)
-        )
-      )
-    )
-  )
-  (symbol (lib_id "Connector:Screw_Terminal_01x04") (at 25.4 54.61 180) (unit 1)
-    (in_bom yes) (on_board yes) (dnp no) (fields_autoplaced)
-    (property "Reference" "J1" (at 25.4 44.45 0)
-      (effects (font (size 1.27 1.27)))
-    )
-    (property "Value" "Screw_Terminal_01x04" (at 25.4 46.99 0)
-      (effects (font (size 1.27 1.27)))
-    )
-    (property "Footprint" "TerminalBlock_Phoenix:TerminalBlock_Phoenix_MKDS-1,5-4-5.08_1x04_P5.08mm_Horizontal" (at 25.4 54.61 0)
-      (effects (font (size 1.27 1.27)) hide)
-    )
-    (property "Datasheet" "~" (at 25.4 54.61 0)
-      (effects (font (size 1.27 1.27)) hide)
-    )
-    (pin "1")
-    (pin "2")
-    (pin "3")
-    (pin "4")
-    (instances
-      (project "LAS_V2"
-        (path "/aadef4b8-3115-4a49-998f-828f2021a6b4"
-          (reference "J1") (unit 1)
         )
       )
@@
       (effects (font (size 1.27 1.27)) (justify right))
     )
-    (property "Footprint" "Connector_PinHeader_1.27mm:PinHeader_1x02_P1.27mm_Vertical" (at 181.61 140.97 0)
+    (property "Footprint" "Connector_PinHeader_2.54mm:PinHeader_1x02_P2.54mm_Vertical" (at 181.61 140.97 0)
       (effects (font (size 1.27 1.27)) hide)
     )
@@
       (effects (font (size 1.27 1.27)))
     )
-    (property "Footprint" "Connector_PinHeader_1.27mm:PinHeader_1x03_P1.27mm_Vertical" (at 26.67 26.67 0)
+    (property "Footprint" "Connector_PinHeader_2.54mm:PinHeader_1x03_P2.54mm_Vertical" (at 26.67 26.67 0)
       (effects (font (size 1.27 1.27)) hide)
     )
@@
       (effects (font (size 1.27 1.27)) (justify left))
     )
-    (property "Footprint" "Connector_PinHeader_1.27mm:PinHeader_1x02_P1.27mm_Vertical" (at 257.81 17.78 0)
+    (property "Footprint" "Connector_PinHeader_2.54mm:PinHeader_1x02_P2.54mm_Vertical" (at 257.81 17.78 0)
       (effects (font (size 1.27 1.27)) hide)
     )
@@
       (effects (font (size 1.27 1.27)) (justify left))
     )
-    (property "Footprint" "Connector_PinHeader_1.27mm:PinHeader_1x22_P1.27mm_Vertical" (at 269.24 135.89 0)
+    (property "Footprint" "Connector_PinHeader_2.54mm:PinHeader_1x22_P2.54mm_Vertical" (at 269.24 135.89 0)
       (effects (font (size 1.27 1.27)) hide)
     )
@@
       (effects (font (size 1.27 1.27)) (justify left top))
     )
-    (pin "VBus" input (at 106.68 110.49 0)
-      (effects (font (size 1.27 1.27)) (justify right))
-    )
     (pin "+3.3V" input (at 78.74 110.49 180)
