File: PCB/LAS_V2/LEDs.kicad_sch (KiCad schematic)
At the start: 7 parts

Commit message: Final Changes to PCB, more code for gateway
Parts:
- added D9: WS2812B, LED_SMD:LED_WS2812B_PLCC4_5.0x5.0mm_P3.2mm, symbol LED:WS2812B
Connections:
- net +5V: now also D9.1 (VDD)
- net GND: now also D9.3 (VSS)
- net at D4.2 (DOUT): now also D9.4 (DIN)
Changed lines of the file:
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@@
   (junction (at 140.97 96.52) (diameter 0) (color 0 0 0 0)
   )
-  (no_connect (at 148.59 116.84))
-  (wire (pts (xy 139.7 127) (xy 139.7 125.73))
-    (stroke (width 0) (type default))
-  )
+  (junction (at 140.97 107.95) (diameter 0) (color 0 0 0 0)
+  )
+  (no_connect (at 170.18 116.84))
   (wire (pts (xy 123.19 107.95) (xy 140.97 107.95))
     (stroke (width 0) (type default))
@@
     (stroke (width 0) (type default))
   )
+  (wire (pts (xy 162.56 107.95) (xy 162.56 109.22))
+    (stroke (width 0) (type default))
+  )
   (wire (pts (xy 160.02 83.82) (xy 160.02 85.09))
     (stroke (width 0) (type default))
@@
     (stroke (width 0) (type default))
   )
-  (wire (pts (xy 140.97 124.46) (xy 140.97 127))
+  (wire (pts (xy 162.56 128.27) (xy 162.56 124.46))
+    (stroke (width 0) (type default))
+  )
+  (wire (pts (xy 140.97 107.95) (xy 162.56 107.95))
+    (stroke (width 0) (type default))
+  )
+  (wire (pts (xy 140.97 124.46) (xy 140.97 128.27))
     (stroke (width 0) (type default))
   )
@@
     (stroke (width 0) (type default))
   )
-  (wire (pts (xy 140.97 127) (xy 139.7 127))
+  (wire (pts (xy 154.94 116.84) (xy 148.59 116.84))
     (stroke (width 0) (type default))
   )
@@
     )
   )
-  (symbol (lib_id "power:GND") (at 139.7 125.73 0) (unit 1)
-    (in_bom yes) (on_board yes) (dnp no) (fields_autoplaced)
-    (property "Reference" "#PWR021" (at 139.7 132.08 0)
-      (effects (font (size 1.27 1.27)) hide)
-    )
-    (property "Value" "GND" (at 139.7 130.81 0)
-      (effects (font (size 1.27 1.27)))
-    )
-    (property "Footprint" "" (at 139.7 125.73 0)
-      (effects (font (size 1.27 1.27)) hide)
-    )
-    (property "Datasheet" "" (at 139.7 125.73 0)
+  (symbol (lib_id "power:GND") (at 140.97 128.27 0) (unit 1)
+    (in_bom yes) (on_board yes) (dnp no) (fields_autoplaced)
+    (property "Reference" "#PWR021" (at 140.97 134.62 0)
+      (effects (font (size 1.27 1.27)) hide)
+    )
+    (property "Value" "GND" (at 140.97 133.35 0)
+      (effects (font (size 1.27 1.27)))
+    )
+    (property "Footprint" "" (at 140.97 128.27 0)
+      (effects (font (size 1.27 1.27)) hide)
+    )
+    (property "Datasheet" "" (at 140.97 128.27 0)
       (effects (font (size 1.27 1.27)) hide)
     )
@@
   (symbol (lib_id "LED:WS2812B") (at 140.97 116.84 0) (unit 1)
     (in_bom yes) (on_board yes) (dnp no)
-    (property "Reference" "D4" (at 154.686 110.49 0)
-      (effects (font (size 1.27 1.27)))
-    )
-    (property "Value" "WS2812B" (at 154.686 113.03 0)
+    (property "Reference" "D4" (at 147.32 106.68 0)
+      (effects (font (size 1.27 1.27)))
+    )
+    (property "Value" "WS2812B" (at 147.32 109.22 0)
       (effects (font (size 1.27 1.27)))
     )
@@
         )
       )
+    )
+  )
+  (symbol (lib_id "power:GND") (at 162.56 128.27 0) (unit 1)
+    (in_bom yes) (on_board yes) (dnp no) (fields_autoplaced)
+    (property "Reference" "#PWR021" (at 162.56 134.62 0)
+      (effects (font (size 1.27 1.27)) hide)
+    )
+    (property "Value" "GND" (at 162.56 133.35 0)
+      (effects (font (size 1.27 1.27)))
+    )
+    (property "Footprint" "" (at 162.56 128.27 0)
+      (effects (font (size 1.27 1.27)) hide)
+    )
+    (property "Datasheet" "" (at 162.56 128.27 0)
+      (effects (font (size 1.27 1.27)) hide)
+    )
+    (pin "1")
+    (instances
+      (project "LAS_V2"
+        (path "/aadef4b8-3115-4a49-998f-828f2021a6b4"
+          (reference "#PWR021") (unit 1)
+        )
+        (path "/aadef4b8-3115-4a49-998f-828f2021a6b4/f48c28f3-4e7e-4446-924c-0b87434ade9c"
+          (reference "#PWR027") (unit 1)
+        )
+      )
+    )
+  )
+  (symbol (lib_id "LED:WS2812B") (at 162.56 116.84 0) (unit 1)
+    (in_bom yes) (on_board yes) (dnp no)
+    (property "Reference" "D9" (at 168.91 106.68 0)
+      (effects (font (size 1.27 1.27)))
+    )
+    (property "Value" "WS2812B" (at 168.91 109.22 0)
+      (effects (font (size 1.27 1.27)))
+    )
+    (property "Footprint" "LED_SMD:LED_WS2812B_PLCC4_5.0x5.0mm_P3.2mm" (at 163.83 124.46 0)
+      (effects (font (size 1.27 1.27)) (justify left top) hide)
+    )
+    (property "Datasheet" "https://cdn-shop.adafruit.com/datasheets/WS2812B.pdf" (at 165.1 126.365 0)
+      (effects (font (size 1.27 1.27)) (justify left top) hide)
+    )
+    (property "LCSC" "C2843785" (at 162.56 116.84 0)
+      (effects (font (size 1.27 1.27)) hide)
+    )
+    (pin "1")
+    (pin "2")
+    (pin "3")
+    (pin "4")
+    (instances
+      (project "LAS_V2"
+        (path "/aadef4b8-3115-4a49-998f-828f2021a6b4/f48c28f3-4e7e-4446-924c-0b87434ade9c"
+          (reference "D9") (unit 1)
+        )
+      )
