File: PCB/LAS_V2/Relay_Controls.kicad_sch (KiCad schematic)
At the start: 7 parts, among them J9 Conn_01x02_Pin, K1 SRD-05VDC-SL-C, Q6 MMBT2222A

Commit message: Final Changes to PCB, more code for gateway
Parts:
- J9: footprint Connector_PinHeader_1.27mm:PinHeader_1x02_P1.27mm_Vertical -> Connector_PinHeader_2.54mm:PinHeader_1x02_P2.54mm_Vertical
Changed lines of the file:
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@@
       (effects (font (size 1.27 1.27)) (justify right))
     )
-    (property "Footprint" "Connector_PinHeader_1.27mm:PinHeader_1x02_P1.27mm_Vertical" (at 93.98 73.66 0)
+    (property "Footprint" "Connector_PinHeader_2.54mm:PinHeader_1x02_P2.54mm_Vertical" (at 93.98 73.66 0)
       (effects (font (size 1.27 1.27)) hide)
     )
