File: PCB/LAS_V2/USB_interface.kicad_sch (KiCad schematic)
At the start: 13 parts, among them J7 USB_C_Receptacle_USB2.0, J8 Conn_01x05, Q2 MMBT2222A, Q3 MMBT2222A, U3 CH340C

Commit message: Need to redo PCB again
Connections:
- net +3.3V: no longer U3.16 (VCC)
- net VBus: now also U3.16 (VCC)

Commit message: Final Changes to PCB, more code for gateway
Parts:
- removed C8: 1uF, Capacitor_SMD:C_0603_1608Metric, symbol Device:C_Small
Connections:
- net +3.3V: now also U3.16 (VCC), U3.4 (V3)
- net VBus renamed VCC_5V
- net VCC_5V: no longer U3.16 (VCC)
Changed lines of the file:
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@@
   (junction (at 101.6 67.31) (diameter 0) (color 0 0 0 0)
   )
-  (junction (at 109.22 53.34) (diameter 0) (color 0 0 0 0)
-  )
   (junction (at 116.84 53.34) (diameter 0) (color 0 0 0 0)
   )
@@
   )
   (junction (at 200.66 111.76) (diameter 0) (color 0 0 0 0)
+  )
+  (junction (at 167.64 49.53) (diameter 0) (color 0 0 0 0)
   )
   (no_connect (at 101.6 83.82))
@@
     (stroke (width 0) (type default))
   )
-  (wire (pts (xy 109.22 53.34) (xy 116.84 53.34))
+  (wire (pts (xy 101.6 53.34) (xy 116.84 53.34))
     (stroke (width 0) (type default))
   )
@@
     (stroke (width 0) (type default))
   )
-  (wire (pts (xy 161.29 49.53) (xy 161.29 52.07))
-    (stroke (width 0) (type default))
-  )
-  (wire (pts (xy 167.64 52.07) (xy 167.64 48.26))
+  (wire (pts (xy 165.1 49.53) (xy 165.1 52.07))
+    (stroke (width 0) (type default))
+  )
+  (wire (pts (xy 167.64 52.07) (xy 167.64 49.53))
+    (stroke (width 0) (type default))
+  )
+  (wire (pts (xy 167.64 49.53) (xy 167.64 44.45))
     (stroke (width 0) (type default))
   )
@@
     (stroke (width 0) (type default))
   )
+  (wire (pts (xy 165.1 49.53) (xy 167.64 49.53))
+    (stroke (width 0) (type default))
+  )
   (wire (pts (xy 250.19 52.07) (xy 242.57 52.07))
     (stroke (width 0) (type default))
@@
     (stroke (width 0) (type default))
   )
-  (wire (pts (xy 161.29 52.07) (xy 165.1 52.07))
-    (stroke (width 0) (type default))
-  )
   (wire (pts (xy 86.36 91.44) (xy 86.36 93.98))
     (stroke (width 0) (type default))
@@
     (stroke (width 0) (type default))
   )
-  (wire (pts (xy 109.22 50.8) (xy 109.22 53.34))
-    (stroke (width 0) (type default))
-  )
   (wire (pts (xy 157.48 64.77) (xy 135.89 64.77))
     (stroke (width 0) (type default))
@@
   )
   (wire (pts (xy 242.57 64.77) (xy 242.57 67.31))
-    (stroke (width 0) (type default))
-  )
-  (wire (pts (xy 101.6 53.34) (xy 109.22 53.34))
     (stroke (width 0) (type default))
   )
@@
     (effects (font (size 1.27 1.27)) (justify left))
   )
+  (hierarchical_label "+3.3V" (shape input) (at 167.64 44.45 90) (fields_autoplaced)
+    (effects (font (size 1.27 1.27)) (justify left))
+  )
   (hierarchical_label "CHIP_PU" (shape input) (at 215.9 111.76 0) (fields_autoplaced)
     (effects (font (size 1.27 1.27)) (justify left))
@@
     (effects (font (size 1.27 1.27)) (justify left))
   )
-  (hierarchical_label "VBus" (shape input) (at 116.84 80.01 90) (fields_autoplaced)
-    (effects (font (size 1.27 1.27)) (justify left))
-  )
   (hierarchical_label "CHIP_PU" (shape input) (at 250.19 52.07 0) (fields_autoplaced)
     (effects (font (size 1.27 1.27)) (justify left))
@@
     (effects (font (size 1.27 1.27)) (justify left))
   )
-  (hierarchical_label "VBus" (shape input) (at 109.22 50.8 90) (fields_autoplaced)
-    (effects (font (size 1.27 1.27)) (justify left))
-  )
-  (hierarchical_label "VCC_5V" (shape input) (at 167.64 48.26 90) (fields_autoplaced)
-    (effects (font (size 1.27 1.27)) (justify left))
-  )
   (hierarchical_label "TXD0" (shape input) (at 121.92 80.01 90) (fields_autoplaced)
+    (effects (font (size 1.27 1.27)) (justify left))
+  )
+  (hierarchical_label "VCC_5V" (shape input) (at 116.84 80.01 90) (fields_autoplaced)
     (effects (font (size 1.27 1.27)) (justify left))
   )
@@
         (path "/aadef4b8-3115-4a49-998f-828f2021a6b4/a475df9f-c6e9-4f77-bf99-c031d1147f10"
           (reference "R12") (unit 1)
-        )
-      )
-    )
-  )
-  (symbol (lib_id "Device:C_Small") (at 161.29 46.99 0) (unit 1)
-    (in_bom yes) (on_board yes) (dnp no)
-    (property "Reference" "C8" (at 154.94 45.72 0)
-      (effects (font (size 1.27 1.27)) (justify left))
-    )
-    (property "Value" "1uF" (at 154.94 48.26 0)
-      (effects (font (size 1.27 1.27)) (justify left))
-    )
-    (property "Footprint" "Capacitor_SMD:C_0603_1608Metric" (at 161.29 46.99 0)
-      (effects (font (size 1.27 1.27)) hide)
-    )
-    (property "Datasheet" "~" (at 161.29 46.99 0)
-      (effects (font (size 1.27 1.27)) hide)
-    )
-    (property "LCSC" "C15849" (at 161.29 46.99 0)
-      (effects (font (size 1.27 1.27)) hide)
-    )
-    (pin "1")
-    (pin "2")
-    (instances
-      (project "LAS_V2"
-        (path "/aadef4b8-3115-4a49-998f-828f2021a6b4/a475df9f-c6e9-4f77-bf99-c031d1147f10"
-          (reference "C8") (unit 1)
         )
       )
@@
         )
       )
-    )
-  )
-  (symbol (lib_id "power:GND") (at 161.29 44.45 180) (unit 1)
-    (in_bom yes) (on_board yes) (dnp no) (fields_autoplaced)
-    (property "Reference" "#PWR023" (at 161.29 38.1 0)
-      (effects (font (size 1.27 1.27)) hide)
-    )
-    (property "Value" "GND" (at 161.29 40.64 0)
-      (effects (font (size 1.27 1.27)))
-    )
-    (property "Footprint" "" (at 161.29 44.45 0)
-      (effects (font (size 1.27 1.27)) hide)
-    )
-    (property "Datasheet" "" (at 161.29 44.45 0)
-      (effects (font (size 1.27 1.27)) hide)
-    )
-    (pin "1")
-    (instances
-      (project "LAS_V2"
-        (path "/aadef4b8-3115-4a49-998f-828f2021a6b4/a475df9f-c6e9-4f77-bf99-c031d1147f10"
-          (reference "#PWR023") (unit 1)
-        )
-      )
